Commit message: Create new wheels for helping stabilization.

File: ugv_assign_description/urdf/bicycle_robot.urdf (robot description, URDF)
Before this commit: robot bicycle_robot, 6 links, 5 joints
Links:
- added link back_body, mass 30; collision mesh filename=package://ugv_assign_description/meshes/Back_Body.stl; visual mesh filename=package://ugv_assign_description/meshes/Back_Body.stl
- added link middle_body, mass 15; collision mesh filename=package://ugv_assign_description/meshes/Mini_Wheels_Body.stl; visual mesh filename=package://ugv_assign_description/meshes/Mini_Wheels_Body.stl
- added link middle_suspension_left, mass 15; collision mesh filename=package://ugv_assign_description/meshes/Middle_Suspension.s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; visual mesh filename=package://ugv_assign_description/meshes/Middle_Suspension.s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
- added link middle_suspension_right, mass 1; collision mesh filename=package://ugv_assign_description/meshes/Middle_Suspension.s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; visual mesh filename=package://ugv_assign_description/meshes/Middle_Suspension.s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
- added link middle_wheel_left, mass 5; collision mesh filename=package://ugv_assign_description/meshes/Mini_Wheels.stl; visual mesh filename=package://ugv_assign_description/meshes/Mini_Wheels.stl
- added link middle_wheel_right, mass 5; collision mesh filename=package://ugv_assign_description/meshes/Mini_Wheels.stl; visual mesh filename=package://ugv_assign_description/meshes/Mini_Wheels.stl
- link body: mass 26.7275394 -> 80
- link front_suspension: mass 2.06456521 -> 7.78054865
- link front_wheel: mass 118.44376142 -> 12
- link rear_wheel: mass 118.44376142 -> 12
Joints:
- added joint back_body_joint: type fixed, parent body, child back_body, origin xyz=0 0 0 rpy=0 0 0
- added joint middle_body_joint: type fixed, parent body, child middle_body, origin xyz=0 0 0 rpy=0 0 0
- added joint middle_suspension_left_joint: type fixed, parent body, child middle_suspension_left, origin xyz=0 0 0 rpy=0 0 3.141592654
- added joint middle_suspension_right_joint: type fixed, parent middle_body, child middle_suspension_right, origin xyz=0 0 0 rpy=0 0 0
- added joint middle_wheel_left_joint: type continuous, parent middle_suspension_left, child middle_wheel_left, origin xyz=0 -0.275 -0.22 rpy=0 0 0, axis 0 1 0
- added joint middle_wheel_right_joint: type continuous, parent middle_suspension_right, child middle_wheel_right, origin xyz=0 -0.275 -0.22 rpy=0 0 0, axis 0 1 0
- joint front_suspension_joint: axis (none) -> 0 0 1; limit (none) -> lower=0.0 upper=0.165 effort=50.0 velocity=1.0; origin xyz=0.00840278 0.0 -0.47161173 rpy=0 0 0 -> xyz=0.00717323 0.0 -0.45356114 rpy=0 0 0; type fixed -> prismatic
- joint front_wheel_joint: origin xyz=0.05422176 0 -0.15074257 rpy=0 0.436549886 0 -> xyz=0.05546002 0 -0.16877486 rpy=0 0.436549886 0
- joint handlebars_joint: limit lower=-0.5 upper=0.5 effort=50.0 velocity=25.0 -> lower=-0.5 upper=0.5 effort=10.0 velocity=5.0
- joint rear_wheel_joint: parent body -> back_body

Commit message: Add camera support. Add Zed Camera. Add IMU Sensor. Start LiDAR sensor.

File: ugv_assign_description/urdf/bicycle_robot.urdf (robot description, URDF)
Before this commit: robot bicycle_robot, 12 links, 11 joints
Links:
- added link camera_stereo; collision mesh filename=package://ugv_assign_description/meshes/Camera_Stereo.stl; visual mesh filename=package://ugv_assign_description/meshes/Camera_Stereo.stl
- added link camera_stereo_left
- added link camera_stereo_right
- added link camera_support, mass 3.4016517; collision mesh filename=package://ugv_assign_description/meshes/Camera_Support.stl; visual mesh filename=package://ugv_assign_description/meshes/Camera_Support.stl
- added link imu_link
Joints:
- added joint camera_stereo_joint: type fixed, parent camera_support, child camera_stereo, origin xyz=0.15649823 0.08 0.09515994 rpy=0 0.436549886 0
- added joint camera_stereo_left_joint: type fixed, parent camera_stereo, child camera_stereo_left, origin xyz=0 0 0 rpy=0 0 0
- added joint camera_stereo_right_joint: type fixed, parent camera_stereo, child camera_stereo_right, origin xyz=0 -0.16 0 rpy=0 0 0
- added joint camera_support_joint: type fixed, parent handlebars, child camera_support, origin xyz=0 0 0 rpy=0 0 0
- added joint imu_joint: type fixed, parent body, child imu_link, origin xyz=0 0 0 rpy=0 0 0

Commit message: Copy the dedesert world. Create joint publishers, imu, laser and camera.

File: ugv_assign_description/urdf/bicycle_robot.urdf (robot description, URDF)
Before this commit: robot bicycle_robot, 17 links, 16 joints
Links:
- added link bicycle_velodyne
- link rear_wheel: mass 12 -> 20
Joints:
- added joint bicycle_velodyne: type fixed, parent body, child bicycle_velodyne, origin xyz=0 0 0 rpy=0 0 0
- joint middle_suspension_left_joint: axis (none) -> 0 0 1; limit (none) -> lower=0.0 upper=0.05 effort=50.0 velocity=1.0; type fixed -> prismatic
- joint middle_suspension_right_joint: axis (none) -> 0 0 1; limit (none) -> lower=0.0 upper=0.05 effort=50.0 velocity=0.1; type fixed -> prismatic
